Commit message: add wrist control (havent tested)

File: robots/demohand/urdf/Demo_urdf_v1.urdf (robot description, URDF)
Before this commit: robot Demo_urdf_v1, 16 links, 15 joints
Links:
- link base_link: geometry collision mesh filename=../meshes/base_link.STL; visual mesh filename=./robots/demohand/meshes/base_link.STL

Commit message: connect slider and 3d model

File: robots/demohand/urdf/Demo_urdf_v1.urdf (robot description, URDF)
Before this commit: robot Demo_urdf_v1, 16 links, 15 joints
Joints:
- removed joint joint1_1
- removed joint joint1_2
- removed joint joint1_3
- removed joint joint2_1
- removed joint joint2_2
- removed joint joint2_3
- removed joint joint3_1
- removed joint joint3_2
- removed joint joint4_1
- removed joint joint4_2
- removed joint joint4_3
- removed joint joint5_1
- removed joint joint5_2
- removed joint joint5_3
- removed joint jonit3_3
- added joint index_dip: type revolute, parent link4_2, child link4_3, origin xyz=-0.03 0 -0.0002 rpy=0 0 0, axis 0 0 -1, limit lower=0 upper=1.39 effort=100 velocity=10
- added joint index_mcp: type revolute, parent base_link, child link4_1, origin xyz=-0.3328 0.026315 0.024636 rpy=1.5708 0 0, axis 0 0 -1, limit lower=0 upper=1.22 effort=100 velocity=10
- added joint index_pip: type revolute, parent link4_1, child link4_2, origin xyz=-0.03359 0 -0.0026 rpy=0 0 0, axis 0 0 -1, limit lower=0 upper=1.39 effort=100 velocity=10
- added joint middle_dip: type revolute, parent link3_2, child link3_3, origin xyz=-0.03 0 -0.0038 rpy=0 0 0, axis 0 0 -1, limit lower=0 upper=1.39 effort=100 velocity=10
- added joint middle_mcp: type revolute, parent base_link, child link3_1, origin xyz=-0.34286 0.0013152 0.024636 rpy=1.5708 0 0, axis 0 0 -1, limit lower=0 upper=1.22 effort=100 velocity=10
- added joint middle_pip: type revolute, parent link3_1, child link3_2, origin xyz=-0.03359 0 -0.0026 rpy=0 0 0, axis 0 0 -1, limit lower=0 upper=1.39 effort=100 velocity=10
- added joint pinky_dip: type revolute, parent link1_2, child link1_3, origin xyz=-0.03 0 -0.0047 rpy=0 0 0, axis 0 0 -1, limit lower=0 upper=1.39 effort=100 velocity=10
- added joint pinky_mcp: type revolute, parent base_link, child link1_1, origin xyz=-0.32226 -0.052285 0.024636 rpy=1.5708 0 0, axis 0 0 -1, limit lower=0 upper=1.22 effort=100 velocity=10
- added joint pinky_pip: type revolute, parent link1_1, child link1_2, origin xyz=-0.03359 0 -0.0017 rpy=0 0 0, axis 0 0 -1, limit lower=0 upper=1.39 effort=100 velocity=10
- added joint ring_dip: type revolute, parent link2_2, child link2_3, origin xyz=-0.03 0 -0.0049 rpy=0 0 0, axis 0 0 -1, limit lower=0 upper=1.39 effort=100 velocity=10
- added joint ring_mcp: type revolute, parent base_link, child link2_1, origin xyz=-0.33407 -0.023685 0.024636 rpy=1.5708 0 0, axis 0 0 -1, limit lower=0 upper=1.22 effort=100 velocity=10
- added joint ring_pip: type revolute, parent link2_1, child link2_2, origin xyz=-0.03359 0 -0.0015 rpy=0 0 0, axis 0 0 -1, limit lower=0 upper=1.39 effort=100 velocity=10
- added joint thumb_cmc: type revolute, parent base_link, child link5_1, origin xyz=-0.27277 0.022223 0.044042 rpy=3.1416 0.61087 0, axis 0 0 -1, limit lower=0 upper=1.22 effort=100 velocity=10
- added joint thumb_ip: type revolute, parent link5_2, child link5_3, origin xyz=-0.03 0 -0.0002 rpy=0 0 0, axis 0 0 -1, limit lower=0 upper=1.39 effort=100 velocity=10
- added joint thumb_mcp: type revolute, parent link5_1, child link5_2, origin xyz=-0.03359 0 -0.0026 rpy=0 0 0, axis 0 0 -1, limit lower=0 upper=1.39 effort=100 velocity=10
