Commit message: add calibrate light; add UDE teleop

File: robots/model3_description_2/model3_urdf.urdf (robot description, URDF)
Before this commit: robot model3, 21 links, 20 joints
Links:
- link base_link: geometry collision mesh filename=./meshes/base_link.fbx scale=0.001 0.001 0.001; visual mesh filename=./meshes/base_link.fbx scale=0.001 0.001 0.001
- link forearm_shell: geometry collision mesh filename=./meshes/forearm_shell.fbx scale=0.001 0.001 0.001; visual mesh filename=./meshes/forearm_shell.fbx scale=0.001 0.001 0.001
- link hand_shell: geometry collision mesh filename=./meshes/hand_shell.fbx scale=0.001 0.001 0.001; visual mesh filename=./meshes/hand_shell.fbx scale=0.001 0.001 0.001
- link hand_skeleton: geometry collision mesh filename=./meshes/hand_skeleton.fbx scale=0.001 0.001 0.001; visual mesh filename=./meshes/hand_skeleton.fbx scale=0.001 0.001 0.001
- link index_dip: geometry collision mesh filename=./meshes/index_dip.fbx scale=0.001 0.001 0.001; visual mesh filename=./meshes/index_dip.fbx scale=0.001 0.001 0.001
- link index_pip: geometry collision mesh filename=./meshes/index_pip.fbx scale=0.001 0.001 0.001; visual mesh filename=./meshes/index_pip.fbx scale=0.001 0.001 0.001
- link index_tip: geometry collision mesh filename=./meshes/index_tip.fbx scale=0.001 0.001 0.001; visual mesh filename=./meshes/index_tip.fbx scale=0.001 0.001 0.001
- link middle_dip: geometry collision mesh filename=./meshes/middle_dip.fbx scale=0.001 0.001 0.001; visual mesh filename=./meshes/middle_dip.fbx scale=0.001 0.001 0.001
- link middle_pip: geometry collision mesh filename=./meshes/middle_pip.fbx scale=0.001 0.001 0.001; visual mesh filename=./meshes/middle_pip.fbx scale=0.001 0.001 0.001
- link middle_tip: geometry collision mesh filename=./meshes/middle_tip.fbx scale=0.001 0.001 0.001; visual mesh filename=./meshes/middle_tip.fbx scale=0.001 0.001 0.001
- link pinky_dip: geometry collision mesh filename=./meshes/pinky_dip.fbx scale=0.001 0.001 0.001; visual mesh filename=./meshes/pinky_dip.fbx scale=0.001 0.001 0.001
- link pinky_pip: geometry collision mesh filename=./meshes/pinky_pip.fbx scale=0.001 0.001 0.001; visual mesh filename=./meshes/pinky_pip.fbx scale=0.001 0.001 0.001
- link pinky_tip: geometry collision mesh filename=./meshes/pinky_tip.fbx scale=0.001 0.001 0.001; visual mesh filename=./meshes/pinky_tip.fbx scale=0.001 0.001 0.001
- link ring_dip: geometry collision mesh filename=./meshes/ring_dip.fbx scale=0.001 0.001 0.001; visual mesh filename=./meshes/ring_dip.fbx scale=0.001 0.001 0.001
- link ring_pip: geometry collision mesh filename=./meshes/ring_pip.fbx scale=0.001 0.001 0.001; visual mesh filename=./meshes/ring_pip.fbx scale=0.001 0.001 0.001
- link ring_tip: geometry collision mesh filename=./meshes/ring_tip.fbx scale=0.001 0.001 0.001; visual mesh filename=./meshes/ring_tip.fbx scale=0.001 0.001 0.001
- link thumb_dip: geometry collision mesh filename=./meshes/thumb_dip.fbx scale=0.001 0.001 0.001; visual mesh filename=./meshes/thumb_dip.fbx scale=0.001 0.001 0.001
- link thumb_pip: geometry collision mesh filename=./meshes/thumb_pip.fbx scale=0.001 0.001 0.001; visual mesh filename=./meshes/thumb_pip.fbx scale=0.001 0.001 0.001
- link thumb_root: geometry collision mesh filename=./meshes/thumb_root.fbx scale=0.001 0.001 0.001; visual mesh filename=./meshes/thumb_root.fbx scale=0.001 0.001 0.001
- link thumb_tip: geometry collision mesh filename=./meshes/thumb_tip.fbx scale=0.001 0.001 0.001; visual mesh filename=./meshes/thumb_tip.fbx scale=0.001 0.001 0.001
- link yaw_pitch_rotor: geometry collision mesh filename=./meshes/yaw_pitch_rotor.fbx scale=0.001 0.001 0.001; visual mesh filename=./meshes/yaw_pitch_rotor.fbx scale=0.001 0.001 0.001
